File: QO100_SPK_ctrl.kicad_pcb (KiCad board)
At the start: 2 copper layers, 67.3 x 41.9 mm, 21 parts, among them J1 PTT in, J2 SPK in, J3 SPK out, J4 12V in, J5 PTT UpConv, J6 PTT ctrl, J7 SPK ctrl, K1 SDS_S2, Q1 BC557B, Q2 BC557B

Commit message: Re-add drill holes for mounting
Parts:
- added REF**: MountingHole_3.2mm_M3_DIN965_Pad, MountingHole:MountingHole_3.2mm_M3_DIN965_Pad, F.Cu at (41.0, 72.0)
- added REF**: MountingHole_3.2mm_M3_DIN965_Pad, MountingHole:MountingHole_3.2mm_M3_DIN965_Pad, F.Cu at (99.9, 72.0)
- added REF**: MountingHole_3.2mm_M3_DIN965_Pad, MountingHole:MountingHole_3.2mm_M3_DIN965_Pad, F.Cu at (99.9, 38.5)
- added REF**: MountingHole_3.2mm_M3_DIN965_Pad, MountingHole:MountingHole_3.2mm_M3_DIN965_Pad, F.Cu at (41.0, 38.5)
Other:
- board text added: "QO-100 SPK Ctrl (c) DF2ET v0.7 02/2022"
- board text removed: "QO-100 SPK Ctrl (c) DF2ET v0.6 01/2022"
